File: AdhanBoxPCBV3/AdhanBoxPCBV3.kicad_pcb (KiCad board)
At the start: 2 copper layers, 77.5 x 52 mm, 42 parts, among them J1 microSD_HC_Hirose_DM3AT-SF-PE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, J2 PinHeader_1x02_P2.54mm_Vertic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, J3 USB_C_Receptacle_HRO_TYPE-C-3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, J4 PinHeader_1x03_P2.54mm_Vertic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, J5 PinHeader_1x03_P2.54mm_Vertic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, J6 PinHeader_1x02_P2.54mm_Vertic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, J7 PinHeader_1x02_P2.54mm_Vertic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, SW1 SW_SPST_TL3342, SW2 SW_SPST_TL3342, U1 ESP32-S3-WROOM-1, U2 QFN-16-1EP_3x3mm_P0.5mm_EP1.4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, U3 SO-14_5.3x10.2mm_P1.27mm, U4 SOT-223-3_TabPin2

Commit message: PCB V3.1 : pont de masse pour l'ampli audio (corrige la saturation)
L'ampli MAX98357A saturait des les cretes alors que la V2, au schema
identique, reste propre. Cause trouvee par analyse comparative des deux
routages : SPK_P et SPK_N sont routees en B.Cu et traversent la carte
(73 et 77 mm ; V2 : 14 mm en F.Cu), ce qui decoupe le plan de masse en
4 ilots. Le GND de U2 se retrouve sur un ruban de 87 mm2 coince ENTRE les
deux sorties commutees, et C1 (100 nF de decouplage) est 0,55 mm au sud de
SPK_N, donc sur un autre ilot : le courant de retour ne peut pas franchir
la piste et fait le tour de la carte.

Boucle de decouplage mesuree : 65-111 mm (V2 de reference : 7-8 mm).
Les condensateurs ne decouplaient donc pas l'ampli, d'ou la distorsion
des que le courant de sortie monte -> saturation au-dela d'un seuil de
volume, insensible a la charge, au chargeur, aux LED et au fichier joue,
avec un rail 5 V pourtant stable a 5,15 V.

Correctif : deux vias en parallele sur le ruban de masse + un saut en
F.Cu par-dessus SPK_N jusqu'a la pastille GND de C1. Boucle ramenee a
6,2 mm, au niveau de la V2. DRC inchange (39 violations preexistantes,
0 critique, 1 ilot de zone).

Co-Authored-By: Claude Fable 5 <noreply@anthropic.com>
Routing:
- net GND: track 0.00 -> 3.01 mm, vias 10 -> 12
Changed lines of the file:
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@@
 	)
 	(embedded_fonts no)
+	(via
+		(at 166 119)
+		(size 0.8)
+		(drill 0.4)
+		(layers "F.Cu" "B.Cu")
+		(net "GND")
+	)
+	(via
+		(at 166.9 119)
+		(size 0.8)
+		(drill 0.4)
+		(layers "F.Cu" "B.Cu")
+		(net "GND")
+	)
+	(segment
+		(start 166.9 119)
+		(end 166 119)
+		(width 1.0)
+		(layer "F.Cu")
+		(net "GND")
+	)
+	(segment
+		(start 166 119)
+		(end 165.5 121.05)
+		(width 1.0)
+		(layer "F.Cu")
+		(net "GND")
+	)
 )
