File: halo/Halo.kicad_pcb (KiCad board)
At the start: 2 copper layers, 85 x 93 mm, 83 parts, among them J1 USB-C 16P, J2 5V / GND alt, Q1 ALS-PT19-315C, SW1 RESET, SW2 BOOT, SW3 USER, U1 ESP32-C3-MINI-1-N4, U2 AMS1117-3.3, U3 74AHCT1G125

Commit message: Halo : le WS2812B-2020 est arrete, bascule sur le WS2812C-2020-V1 ; F1 et U3 references
JLCPCB refusait le devis : F1 sans reference LCSC (son outil cherchait alors la
description en francais, sans resultat) et 118 LEDs manquantes sur 122.

- LED1-LED24 : WS2812B-2020 (C965555) arrete par Worldsemi, 4 en stock. Remplace
  par le WS2812C-2020-V1 (C2976072, 53301 en stock) : meme boitier 2.2 x 2.0,
  meme empreinte au 0.01 mm, meme brochage 1 DO 2 GND 3 DI 4 VDD, verifie sur la
  datasheet. Il tire 5 mA par canal au lieu de 12 : halo moins lumineux, budget
  USB plus large (360 mA en blanc plein au lieu de 860). A juger sur le proto.
- F1 : SMD1206P110TF RUILON (C20801), 1.1 A / 6 V en 1206. Le MF-MSMF110-2 de
  Bourns qui etait cite en note est en 1812, il n'entre pas dans l'empreinte.
- U3 : 74AHCT1G125GV MDD (C52140417), SOT-23-5L, 5183 en stock.
- Le champ Comment de la BOM porte desormais la reference fabricant seule : c'est
  la chaine que JLCPCB envoie dans sa recherche quand il n'a pas de code LCSC.
- SCHEMA.md : budget de puissance, brochage LED et section « a confirmer » refaits.

Chaine rejouee en entier : DRC 0 erreur, BOM, CPL et PCB concordent, plus aucune
reference LCSC manquante.

Co-Authored-By: Claude Opus 5 <noreply@anthropic.com>
Parts:
- LED1, LED10, LED11, LED12, LED13, LED14, LED15, LED16, LED17, LED18, LED19, LED2, LED20, LED21, LED22, LED23, LED24, LED3, LED4, LED5, LED6, LED7, LED8, LED9: value WS2812B-2020 -> WS2812C-2020-V1
Changed lines of the file:
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@@
 			)
 		)
-		(property "Value" "WS2812B-2020"
+		(property "Value" "WS2812C-2020-V1"
 			(at 0 2.1 0)
 			(layer "F.Fab")
@@
 			)
 		)
-		(property "Value" "WS2812B-2020"
+		(property "Value" "WS2812C-2020-V1"
 			(at 0 2.1 0)
 			(layer "F.Fab")
@@
 			)
 		)
-		(property "Value" "WS2812B-2020"
+		(property "Value" "WS2812C-2020-V1"
 			(at 0 2.1 0)
 			(layer "F.Fab")
@@
 			)
 		)
-		(property "Value" "WS2812B-2020"
+		(property "Value" "WS2812C-2020-V1"
 			(at 0 2.1 0)
 			(layer "F.Fab")
@@
 			)
 		)
-		(property "Value" "WS2812B-2020"
+		(property "Value" "WS2812C-2020-V1"
 			(at 0 2.1 0)
 			(layer "F.Fab")
@@
 			)
 		)
-		(property "Value" "WS2812B-2020"
+		(property "Value" "WS2812C-2020-V1"
 			(at 0 2.1 0)
 			(layer "F.Fab")
@@
 			)
 		)
-		(property "Value" "WS2812B-2020"
+		(property "Value" "WS2812C-2020-V1"
 			(at 0 2.1 0)
 			(layer "F.Fab")
@@
 			)
 		)
-		(property "Value" "WS2812B-2020"
+		(property "Value" "WS2812C-2020-V1"
 			(at 0 2.1 0)
 			(layer "F.Fab")
@@
 			)
 		)
-		(property "Value" "WS2812B-2020"
+		(property "Value" "WS2812C-2020-V1"
 			(at 0 2.1 0)
 			(layer "F.Fab")
@@
 			)
 		)
-		(property "Value" "WS2812B-2020"
+		(property "Value" "WS2812C-2020-V1"
 			(at 0 2.1 0)
 			(layer "F.Fab")
@@
 			)
 		)
-		(property "Value" "WS2812B-2020"
+		(property "Value" "WS2812C-2020-V1"
 			(at 0 2.1 0)
 			(layer "F.Fab")
@@
 			)
 		)
-		(property "Value" "WS2812B-2020"
+		(property "Value" "WS2812C-2020-V1"
 			(at 0 2.1 0)
 			(layer "F.Fab")
@@
 			)
 		)
-		(property "Value" "WS2812B-2020"
+		(property "Value" "WS2812C-2020-V1"
 			(at 0 2.1 0)
 			(layer "F.Fab")
@@
 			)
 		)
-		(property "Value" "WS2812B-2020"
+		(property "Value" "WS2812C-2020-V1"
 			(at 0 2.1 0)
 			(layer "F.Fab")
@@
 			)
 		)
-		(property "Value" "WS2812B-2020"
+		(property "Value" "WS2812C-2020-V1"
 			(at 0 2.1 0)
 			(layer "F.Fab")
@@
 			)
 		)
-		(property "Value" "WS2812B-2020"
+		(property "Value" "WS2812C-2020-V1"
 			(at 0 2.1 0)
 			(layer "F.Fab")
@@
 			)
 		)
-		(property "Value" "WS2812B-2020"
+		(property "Value" "WS2812C-2020-V1"
 			(at 0 2.1 0)
 			(layer "F.Fab")
@@
 			)
 		)
-		(property "Value" "WS2812B-2020"
+		(property "Value" "WS2812C-2020-V1"
 			(at 0 2.1 0)
 			(layer "F.Fab")
@@
 			)
 		)
-		(property "Value" "WS2812B-2020"
+		(property "Value" "WS2812C-2020-V1"
 			(at 0 2.1 0)
 			(layer "F.Fab")
@@
 			)
 		)
-		(property "Value" "WS2812B-2020"
+		(property "Value" "WS2812C-2020-V1"
 			(at 0 2.1 0)
 			(layer "F.Fab")
@@
 			)
 		)
-		(property "Value" "WS2812B-2020"
+		(property "Value" "WS2812C-2020-V1"
 			(at 0 2.1 0)
 			(layer "F.Fab")
@@
 			)
 		)
-		(property "Value" "WS2812B-2020"
+		(property "Value" "WS2812C-2020-V1"
 			(at 0 2.1 0)
 			(layer "F.Fab")
@@
 			)
 		)
-		(property "Value" "WS2812B-2020"
+		(property "Value" "WS2812C-2020-V1"
 			(at 0 2.1 0)
 			(layer "F.Fab")
@@
 			)
 		)
-		(property "Value" "WS2812B-2020"
+		(property "Value" "WS2812C-2020-V1"
 			(at 0 2.1 0)
 			(layer "F.Fab")
